File: KiCAD/CounterModule/CounterModule.kicad_pcb (KiCad board)
At the start: 2 copper layers, 68 parts, among them Q1 2N3906, Q10 2N3906, Q11 2N3906, Q12 2N3906, Q13 2N3906, Q14 2N3906, Q15 2N3906, Q16 2N3906, Q17 2N3904, Q18 2N3904, Q19 2N3904, Q2 2N3906, Q3 2N3906, Q4 2N3906, Q5 2N3906, Q6 2N3906, Q7 2N3906, Q8 2N3906, Q9 2N3906

Commit message: attempt at universal counter
Parts:
- added C13: 0.1uF, Capacitor_THT:C_Disc_D4.3mm_W1.9mm_P5.00mm, F.Cu at (61.6, 45.1)
- added C14: 0.1uF, Capacitor_THT:C_Disc_D4.3mm_W1.9mm_P5.00mm, F.Cu at (94.2, 45.2)
- added C15: 0.1uF, Capacitor_THT:C_Disc_D4.3mm_W1.9mm_P5.00mm, F.Cu at (126.9, 45.0)
- added C16: 500p, Capacitor_THT:C_Disc_D4.3mm_W1.9mm_P5.00mm, F.Cu at (68.7, 60.4)
- added C17: 500p, Capacitor_THT:C_Disc_D4.3mm_W1.9mm_P5.00mm, F.Cu at (82.0, 60.4)
- added C18: 500p, Capacitor_THT:C_Disc_D4.3mm_W1.9mm_P5.00mm, F.Cu at (65.5, 63.6)
- added C19: 500p, Capacitor_THT:C_Disc_D4.3mm_W1.9mm_P5.00mm, F.Cu at (102.4, 60.4)
- added C20: 500p, Capacitor_THT:C_Disc_D4.3mm_W1.9mm_P5.00mm, F.Cu at (115.7, 60.4)
- added C21: 500p, Capacitor_THT:C_Disc_D4.3mm_W1.9mm_P5.00mm, F.Cu at (99.2, 63.6)
- added C22: 500p, Capacitor_THT:C_Disc_D4.3mm_W1.9mm_P5.00mm, F.Cu at (134.8, 60.4)
- added C23: 500p, Capacitor_THT:C_Disc_D4.3mm_W1.9mm_P5.00mm, F.Cu at (148.1, 60.4)
- added C24: 500p, Capacitor_THT:C_Disc_D4.3mm_W1.9mm_P5.00mm, F.Cu at (131.6, 63.6)
- added C25: 0.1uF, Capacitor_THT:C_Disc_D4.3mm_W1.9mm_P5.00mm, F.Cu at (159.6, 45.2)
- added C26: 0.1uF, Capacitor_THT:C_Disc_D4.3mm_W1.9mm_P5.00mm, F.Cu at (60.5, 66.8)
- added C27: 0.1uF, Capacitor_THT:C_Disc_D4.3mm_W1.9mm_P5.00mm, F.Cu at (94.2, 66.8)
- added C28: 0.1uF, Capacitor_THT:C_Disc_D4.3mm_W1.9mm_P5.00mm, F.Cu at (126.5, 66.8)
- added D1: 1N4148, Diode_THT:D_DO-35_SOD27_P7.62mm_Horizontal, F.Cu at (178.1, 54.6)
- added D2: 1N4148, Diode_THT:D_DO-35_SOD27_P7.62mm_Horizontal, F.Cu at (178.1, 58.2)
- added JP1: Jumper_2_Open, Connector_PinHeader_2.54mm:PinHeader_1x02_P2.54mm_Vertical, F.Cu at (191.1, 57.1)
- added JP2: Jumper_3_Open, Connector_PinHeader_2.54mm:PinHeader_1x03_P2.54mm_Vertical, F.Cu at (127.0, 71.1)
- added JP3: Jumper_3_Open, Connector_PinHeader_2.54mm:PinHeader_1x03_P2.54mm_Vertical, F.Cu at (127.6, 49.5)
- added Q20: 2N3904, Package_TO_SOT_THT:TO-92_Inline, F.Cu at (162.2, 56.4)
- added Q21: 2N3904, Package_TO_SOT_THT:TO-92_Inline, F.Cu at (162.2, 62.2)
- added Q22: 2N3904, Package_TO_SOT_THT:TO-92_Inline, F.Cu at (162.2, 68.0)
- added Q23: 2N3906, Package_TO_SOT_THT:TO-92_Inline, F.Cu at (53.7, 52.9)
- added Q24: 2N3906, Package_TO_SOT_THT:TO-92_Inline, F.Cu at (53.7, 59.8)
- added Q25: 2N3906, Package_TO_SOT_THT:TO-92_Inline, F.Cu at (53.7, 31.3)
- added Q26: 2N3906, Package_TO_SOT_THT:TO-92_Inline, F.Cu at (53.7, 38.2)
- added Q27: 2N3906, Package_TO_SOT_THT:TO-92_Inline, F.Cu at (62.4, 54.1)
- added Q28: 2N3906, Package_TO_SOT_THT:TO-92_Inline, F.Cu at (71.3, 54.1)
- added Q29: 2N3906, Package_TO_SOT_THT:TO-92_Inline, F.Cu at (79.8, 54.1)
- added Q30: 2N3906, Package_TO_SOT_THT:TO-92_Inline, F.Cu at (87.4, 54.1)
- added Q31: 2N3906, Package_TO_SOT_THT:TO-92_Inline, F.Cu at (96.0, 54.1)
- added Q32: 2N3906, Package_TO_SOT_THT:TO-92_Inline, F.Cu at (104.9, 54.1)
- added Q33: 2N3906, Package_TO_SOT_THT:TO-92_Inline, F.Cu at (113.5, 54.1)
- added Q34: 2N3906, Package_TO_SOT_THT:TO-92_Inline, F.Cu at (121.1, 54.1)
- added Q35: 2N3906, Package_TO_SOT_THT:TO-92_Inline, F.Cu at (128.4, 54.1)
- added Q36: 2N3906, Package_TO_SOT_THT:TO-92_Inline, F.Cu at (137.3, 54.1)
- added Q37: 2N3906, Package_TO_SOT_THT:TO-92_Inline, F.Cu at (145.8, 54.1)
- added Q38: 2N3906, Package_TO_SOT_THT:TO-92_Inline, F.Cu at (153.5, 54.1)
- added R38: 1k, Resistor_THT:R_Axial_DIN0204_L3.6mm_D1.6mm_P2.54mm_Vertical, F.Cu at (168.3, 54.7)
- added R39: 1k, Resistor_THT:R_Axial_DIN0204_L3.6mm_D1.6mm_P2.54mm_Vertical, F.Cu at (168.3, 57.9)
- added R40: 4.7k, Resistor_THT:R_Axial_DIN0204_L3.6mm_D1.6mm_P2.54mm_Vertical, F.Cu at (168.3, 61.0)
- added R41: 4.7k, Resistor_THT:R_Axial_DIN0204_L3.6mm_D1.6mm_P2.54mm_Vertical, F.Cu at (168.3, 64.2)
- added R42: 4.7k, Resistor_THT:R_Axial_DIN0204_L3.6mm_D1.6mm_P2.54mm_Vertical, F.Cu at (168.3, 67.3)
- added R43: 4.7k, Resistor_THT:R_Axial_DIN0204_L3.6mm_D1.6mm_P2.54mm_Vertical, F.Cu at (47.4, 54.1)
- added R44: 4.7k, Resistor_THT:R_Axial_DIN0204_L3.6mm_D1.6mm_P2.54mm_Vertical, F.Cu at (47.4, 61.1)
- added R45: R_US, Resistor_THT:R_Axial_DIN0204_L3.6mm_D1.6mm_P2.54mm_Vertical, F.Cu at (53.7, 65.6)
- added R46: 4.7k, Resistor_THT:R_Axial_DIN0204_L3.6mm_D1.6mm_P2.54mm_Vertical, F.Cu at (47.4, 32.5)
- added R47: 4.7k, Resistor_THT:R_Axial_DIN0204_L3.6mm_D1.6mm_P2.54mm_Vertical, F.Cu at (47.4, 39.5)
- added R48: R_US, Resistor_THT:R_Axial_DIN0204_L3.6mm_D1.6mm_P2.54mm_Vertical, F.Cu at (53.7, 44.0)
- added R51: 4.7k, Resistor_THT:R_Axial_DIN0204_L3.6mm_D1.6mm_P2.54mm_Vertical, F.Cu at (61.2, 60.4)
- added R52: 4.7k, Resistor_THT:R_Axial_DIN0204_L3.6mm_D1.6mm_P2.54mm_Vertical, F.Cu at (87.7, 60.4)
- added R53: 4.7k, Resistor_THT:R_Axial_DIN0204_L3.6mm_D1.6mm_P2.54mm_Vertical, F.Cu at (70.6, 63.6)
- added R54: 4.7k, Resistor_THT:R_Axial_DIN0204_L3.6mm_D1.6mm_P2.54mm_Vertical, F.Cu at (80.7, 63.6)
- added R55: 470, Resistor_THT:R_Axial_DIN0204_L3.6mm_D1.6mm_P2.54mm_Vertical, F.Cu at (70.6, 66.8)
- added R56: 470, Resistor_THT:R_Axial_DIN0204_L3.6mm_D1.6mm_P2.54mm_Vertical, F.Cu at (80.7, 66.8)
- added R57: 1k, Resistor_THT:R_Axial_DIN0204_L3.6mm_D1.6mm_P2.54mm_Vertical, F.Cu at (85.3, 63.6)
- added R58: 470, Resistor_THT:R_Axial_DIN0204_L3.6mm_D1.6mm_P2.54mm_Vertical, F.Cu at (78.3, 69.9)
- added R59: 4.7k, Resistor_THT:R_Axial_DIN0204_L3.6mm_D1.6mm_P2.54mm_Vertical, F.Cu at (94.8, 60.4)
- added R60: 4.7k, Resistor_THT:R_Axial_DIN0204_L3.6mm_D1.6mm_P2.54mm_Vertical, F.Cu at (121.4, 60.4)
- added R61: 4.7k, Resistor_THT:R_Axial_DIN0204_L3.6mm_D1.6mm_P2.54mm_Vertical, F.Cu at (104.2, 63.6)
- added R62: 4.7k, Resistor_THT:R_Axial_DIN0204_L3.6mm_D1.6mm_P2.54mm_Vertical, F.Cu at (114.4, 63.6)
- added R63: 470, Resistor_THT:R_Axial_DIN0204_L3.6mm_D1.6mm_P2.54mm_Vertical, F.Cu at (104.3, 66.8)
- added R64: 470, Resistor_THT:R_Axial_DIN0204_L3.6mm_D1.6mm_P2.54mm_Vertical, F.Cu at (114.4, 66.8)
- added R65: 1k, Resistor_THT:R_Axial_DIN0204_L3.6mm_D1.6mm_P2.54mm_Vertical, F.Cu at (118.9, 63.6)
- added R66: 470, Resistor_THT:R_Axial_DIN0204_L3.6mm_D1.6mm_P2.54mm_Vertical, F.Cu at (112.0, 69.9)
- added R67: 4.7k, Resistor_THT:R_Axial_DIN0204_L3.6mm_D1.6mm_P2.54mm_Vertical, F.Cu at (127.2, 60.4)
- added R68: 4.7k, Resistor_THT:R_Axial_DIN0204_L3.6mm_D1.6mm_P2.54mm_Vertical, F.Cu at (153.8, 60.4)
- added R69: 4.7k, Resistor_THT:R_Axial_DIN0204_L3.6mm_D1.6mm_P2.54mm_Vertical, F.Cu at (136.6, 63.6)
- added R70: 4.7k, Resistor_THT:R_Axial_DIN0204_L3.6mm_D1.6mm_P2.54mm_Vertical, F.Cu at (146.8, 63.6)
- added R71: 470, Resistor_THT:R_Axial_DIN0204_L3.6mm_D1.6mm_P2.54mm_Vertical, F.Cu at (136.7, 66.8)
- added R72: 470, Resistor_THT:R_Axial_DIN0204_L3.6mm_D1.6mm_P2.54mm_Vertical, F.Cu at (146.8, 66.8)
- added R73: 1k, Resistor_THT:R_Axial_DIN0204_L3.6mm_D1.6mm_P2.54mm_Vertical, F.Cu at (151.3, 63.6)
- added R74: 470, Resistor_THT:R_Axial_DIN0204_L3.6mm_D1.6mm_P2.54mm_Vertical, F.Cu at (144.3, 69.9)
- moved R31 87.5 mm to (186.8, 38.8), turned to 180 degrees
- moved R32 85.1 mm to (184.3, 42.0)
- moved Q16 83.3 mm to (186.5, 32.5), turned to -90 degrees
- moved Q3 83.2 mm to (63.5, 32.4), turned to -90 degrees
- moved R29 78.7 mm to (179.8, 42.0), turned to 180 degrees
- moved R30 78.7 mm to (179.8, 45.2), turned to 180 degrees
- moved C3 77.5 mm to (66.6, 41.9), turned to 180 degrees
- moved R6 77.0 mm to (62.3, 38.7)
- moved R28 75.4 mm to (177.4, 48.4)
- moved Q15 74.2 mm to (178.9, 32.5), turned to -90 degrees
- moved C1 73.0 mm to (69.8, 38.7)
- moved Q2 72.6 mm to (72.4, 32.4), turned to -90 degrees
- moved Q4 69.3 mm to (88.5, 32.4), turned to -90 degrees
- moved R27 67.9 mm to (169.6, 42.0)
- moved R26 67.7 mm to (169.7, 45.2)
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Connections:
- R17 pad 1: /CARRY/CY -> /FlipFlop0/RST
- R25 pad 1: /CARRY/CY -> /FlipFlop0/RST
- R6 pad 1: /CARRY/CY -> /FlipFlop0/RST
- R9 pad 1: /CARRY/CY -> /FlipFlop0/RST
Routing:
- net -6V: track 0.00 -> 229.9 mm
- net GND: track 0.00 -> 175.3 mm
- net Net-(Q35-C): track 0.00 -> 20.9 mm
- net Net-(Q2-C): track 0.00 -> 20.9 mm
- net Net-(Q5-C): track 0.00 -> 20.9 mm
- net Net-(Q31-C): track 0.00 -> 20.9 mm
- net Net-(Q27-C): track 0.00 -> 20.9 mm
- net Net-(Q10-C): track 0.00 -> 20.9 mm
- net Net-(Q13-C): track 0.00 -> 20.9 mm
- net Net-(C10-Pad1): track 0.00 -> 17.2 mm
- net Net-(C24-Pad1): track 0.00 -> 17.2 mm
- net Net-(C7-Pad1): track 0.00 -> 17.2 mm
- net Net-(C4-Pad1): track 0.00 -> 17.2 mm
- net Net-(C3-Pad1): track 0.00 -> 17.2 mm
- net Net-(C21-Pad1): track 0.00 -> 17.2 mm
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Other:
- board outline added: 165.1 x 50.8 mm
