File: KiCAD/CounterModule/CounterModule.kicad_sch (KiCad schematic)
At the start: 0 parts

Commit message: attempt at universal counter
Parts:
- added D1, D2: 1N4148, Diode_THT:D_DO-35_SOD27_P7.62mm_Horizontal, symbol Diode:1N4148
- added JP1: Jumper_2_Open, Connector_PinHeader_2.54mm:PinHeader_1x02_P2.54mm_Vertical, symbol Jumper:Jumper_2_Open
- added JP2, JP3: Jumper_3_Open, Connector_PinHeader_2.54mm:PinHeader_1x03_P2.54mm_Vertical, symbol Jumper:Jumper_3_Open
Connections:
- net CARRY/CY: now also D1.1 (K)
- net CARRY/INB: now also JP3.3 (B)
- new net: D2.2 (A), JP1.1 (A)
- new net CARRY1/CY: D2.1 (K)
- new net CARRY1/INA: JP3.2 (C)
- new net CARRY1/INB: JP2.2 (C)
- new net FlipFlop0/RST: D1.2 (A), JP1.2 (B)
- new net FlipFlop5/Q: JP2.1 (A)
- new net FlipFlop6/Q: JP2.3 (B)
- new net FlipFlop7/Q: JP3.1 (A)
Other:
- added sheet CARRY1 (carry.kicad_sch)
- added sheet FlipFlop5 (FlipFlop.kicad_sch)
- added sheet FlipFlop6 (FlipFlop.kicad_sch)
- added sheet FlipFlop7 (FlipFlop.kicad_sch)
- added sheet enable (enable.kicad_sch)
- added sheet enable1 (enable.kicad_sch)
- note added: "1"
- note added: "2"
- note added: "4"
- note added: "8"
- note added: "JP1 in: HOURS out: MIN/SEC"
- note added: "JP2: 1-2 HOURS 2-3 MIN/SEC"
- note added: "JP3: 1-2 MIN/SEC 2-3 HOURS"
- note added: "MIN/SEC 00-59 -or- HOURS 00-23"
