File: KiCAD/CounterModule/FlipFlop.kicad_sch (KiCad schematic)
At the start: 15 parts, among them Q1 2N3906, Q2 2N3906, Q3 2N3906, Q4 2N3906

Commit message: attempt at universal counter
Parts:
- added C13: 0.1uF, Capacitor_THT:C_Disc_D4.3mm_W1.9mm_P5.00mm, symbol Device:C
Connections:
- net -6V: now also C13.2
- net GND: now also C13.1
