File: KiCAD/CounterModule/enable.kicad_sch (KiCad schematic)
At the start: 8 parts, among them Q17 2N3904, Q18 2N3904, Q19 2N3904

Commit message: attempt at universal counter
Parts:
- removed Q17, Q18, Q19: 2N3904, Package_TO_SOT_THT:TO-92_Inline, symbol Transistor_BJT:2N3904
- removed R33, R34, R36: 4.7k, Resistor_THT:R_Axial_DIN0204_L3.6mm_D1.6mm_P2.54mm_Vertical, symbol Device:R_US
- removed R35, R37: 1k, Resistor_THT:R_Axial_DIN0204_L3.6mm_D1.6mm_P2.54mm_Vertical, symbol Device:R_US
- added Q25, Q26: 2N3906, Package_TO_SOT_THT:TO-92_Inline, symbol Transistor_BJT:2N3906
- added R46, R47: 4.7k, Resistor_THT:R_Axial_DIN0204_L3.6mm_D1.6mm_P2.54mm_Vertical, symbol Device:R_US
- added R48: R_US, Resistor_THT:R_Axial_DIN0204_L3.6mm_D1.6mm_P2.54mm_Vertical, symbol Device:R_US
Connections:
- net -6V: now also R48.2
- net GND: now also Q25.1 (E)
- new net: Q26.2 (B), R47.2
- new net: Q25.2 (B), R46.2
- new net: Q25.3 (C), Q26.1 (E)
- new net CLK: Q26.3 (C), R48.1
- new net ENA: R46.1
- new net ~{CLK}: R47.1
